Commit message: URDF file is modified such that all joints' limits from -2*PI to 2*PI are replaced to be from -PI to PI.

File: data/xarm6/xarm6-original.urdf (robot description, URDF)
Before this commit: robot xarm6, 9 links, 8 joints
Joints:
- joint joint1: limit lower=-3.14159265359 upper=3.14159265359 effort=50.0 velocity=3.14 -> lower=-6.28318530718 upper=6.28318530718 effort=50.0 velocity=3.14
- joint joint4: limit lower=-3.14159265359 upper=3.14159265359 effort=32.0 velocity=3.14 -> lower=-6.28318530718 upper=6.28318530718 effort=32.0 velocity=3.14
- joint joint6: limit lower=-3.14159265359 upper=3.14159265359 effort=20.0 velocity=3.14 -> lower=-6.28318530718 upper=6.28318530718 effort=20.0 velocity=3.14
