Commit message: Spatial 14dof, 18dof and 22dof robots and corresponding files created.

File: data/spatial_14dof/spatial_14dof.urdf (robot description, URDF)
Before this commit: robot spatial_10dof, 12 links, 11 joints
Links:
- added link link11, mass 0.1; collision box size=0.05 0.05 0.0692; visual box size=0.05 0.05 0.0692
- added link link12, mass 0.1; collision box size=0.05 0.05 0.0692; visual box size=0.05 0.05 0.0692
- added link link13, mass 0.1; collision box size=0.05 0.05 0.0692; visual box size=0.05 0.05 0.0692
- added link link14, mass 0.1; collision box size=0.05 0.05 0.0692; visual box size=0.05 0.05 0.0692
- link link10: geometry collision box size=0.05 0.05 0.0692; visual box size=0.05 0.05 0.0692
- link link2: geometry collision box size=0.05 0.05 0.0692; visual box size=0.05 0.05 0.0692
- link link3: geometry collision box size=0.05 0.05 0.0692; visual box size=0.05 0.05 0.0692
- link link4: geometry collision box size=0.05 0.05 0.0692; visual box size=0.05 0.05 0.0692
- link link5: geometry collision box size=0.05 0.05 0.0692; visual box size=0.05 0.05 0.0692
- link link6: geometry collision box size=0.05 0.05 0.0692; visual box size=0.05 0.05 0.0692
- link link7: geometry collision box size=0.05 0.05 0.0692; visual box size=0.05 0.05 0.0692
- link link8: geometry collision box size=0.05 0.05 0.0692; visual box size=0.05 0.05 0.0692
- link link9: geometry collision box size=0.05 0.05 0.0692; visual box size=0.05 0.05 0.0692
Joints:
- added joint joint11: type revolute, parent link10, child link11, origin xyz=0 0 0.0692 rpy=0 0 0, axis 1 0 0, limit lower=-3.14159 upper=3.14159 effort=30 velocity=3.14159
- added joint joint12: type revolute, parent link11, child link12, origin xyz=0 0 0.0692 rpy=0 0 0, axis 1 0 0, limit lower=-3.14159 upper=3.14159 effort=30 velocity=3.14159
- added joint joint13: type revolute, parent link12, child link13, origin xyz=0 0 0.0692 rpy=0 0 0, axis 1 0 0, limit lower=-3.14159 upper=3.14159 effort=30 velocity=3.14159
- added joint joint14: type revolute, parent link13, child link14, origin xyz=0 0 0.0692 rpy=0 0 0, axis 1 0 0, limit lower=-3.14159 upper=3.14159 effort=30 velocity=3.14159
- joint ee: origin xyz=0 0 0.1 rpy=0 0 0 -> xyz=0 0 0.0692 rpy=0 0 0; parent link10 -> link14
- joint joint10: origin xyz=0 0 0.1 rpy=0 0 0 -> xyz=0 0 0.0692 rpy=0 0 0
- joint joint3: origin xyz=0 0 0.1 rpy=0 0 0 -> xyz=0 0 0.0692 rpy=0 0 0
- joint joint4: origin xyz=0 0 0.1 rpy=0 0 0 -> xyz=0 0 0.0692 rpy=0 0 0
- joint joint5: origin xyz=0 0 0.1 rpy=0 0 0 -> xyz=0 0 0.0692 rpy=0 0 0
- joint joint6: origin xyz=0 0 0.1 rpy=0 0 0 -> xyz=0 0 0.0692 rpy=0 0 0
- joint joint7: origin xyz=0 0 0.1 rpy=0 0 0 -> xyz=0 0 0.0692 rpy=0 0 0
- joint joint8: origin xyz=0 0 0.1 rpy=0 0 0 -> xyz=0 0 0.0692 rpy=0 0 0
- joint joint9: origin xyz=0 0 0.1 rpy=0 0 0 -> xyz=0 0 0.0692 rpy=0 0 0
